File: Hardwares/MainController/rev2/opsx_x.kicad_sch (KiCad schematic)
At the start: 62 parts, among them J1 Conn_01x02, J3 Conn_01x02, Q1 Q_NMOS_GSD, Q2 Q_NMOS_GSD, Q3 Q_PMOS_GSD, Q4 MMBT3904, U1 RP2040, U2 TLV70433DBVR, U3 W25Q128JVS, U4 OPTICAL-TSL2561T(6P-3.8X2.6MM)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

Commit message: 声纳工作正常
Parts:
- removed D6: LED, Diode_SMD:D_0603_1608Metric_Pad1.05x0.95mm_HandSolder, symbol Device:LED
Changed lines of the file:
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@@
 (kicad_sch
-	(version 20231120)
+	(version 20250114)
 	(generator "eeschema")
-	(generator_version "8.0")
+	(generator_version "9.0")
 	(paper "A3")
 	(title_block
@@
 		(rev "2")
 	)
+	(rectangle
+		(start 13.97 145.415)
+		(end 45.085 187.96)
+		(stroke
+			(width 0)
+			(type default)
+		)
+		(fill
+			(type none)
+		)
+	)
+	(rectangle
+		(start 13.97 13.97)
+		(end 194.31 187.96)
+		(stroke
+			(width 0.3)
+			(type default)
+		)
+		(fill
+			(type none)
+		)
+	)
+	(rectangle
+		(start 13.97 187.96)
+		(end 247.015 282.575)
+		(stroke
+			(width 0)
+			(type default)
+		)
+		(fill
+			(type none)
+		)
+	)
+	(rectangle
+		(start 13.97 122.555)
+		(end 45.085 145.415)
+		(stroke
+			(width 0)
+			(type default)
+		)
+		(fill
+			(type none)
+		)
+	)
+	(text "Flash\n"
+		(exclude_from_sim no)
+		(at 266.7 130.175 0)
+		(effects
+			(font
+				(size 1.27 1.27)
+			)
+			(justify left bottom)
+		)
+	)
+	(text "Meter0"
+		(exclude_from_sim no)
+		(at 257.175 65.405 0)
+		(effects
+			(font
+				(size 1.27 1.27)
+			)
+			(justify left bottom)
+		)
+	)
+	(text "Power "
+		(exclude_from_sim no)
+		(at 38.735 44.45 0)
+		(effects
+			(font
+				(size 1.27 1.27)
+			)
+			(justify left bottom)
+		)
+	)
+	(text "Crystal\n"
+		(exclude_from_sim no)
+		(at 36.83 144.78 0)
+		(effects
+			(font
+				(size 1.27 1.27)
+			)
+			(justify left bottom)
+		)
+	)
+	(text "IF Sonar: high means button got pressed\nELSE : low"
+		(exclude_from_sim no)
+		(at 115.57 198.12 0)
+		(effects
+			(font
+				(size 1.27 1.27)
+			)
+			(justify left bottom)
+		)
+	)
+	(text "Controller (RP2040 )\n"
+		(exclude_from_sim no)
+		(at 147.955 186.055 0)
+		(effects
+			(font
+				(face "KiCad Font")
+				(size 2.54 2.54)
+				(thickness 0.508)
+				(bold yes)
+			)
+			(justify left bottom)
+		)
+	)
+	(text "SCL1\n"
+		(exclude_from_sim no)
+		(at 151.13 139.7 0)
+		(effects
+			(font
+				(size 1.27 1.27)
+			)
+			(justify left bottom)
+		)
+	)
+	(text "SDA1"
+		(exclude_from_sim no)
+		(at 151.13 137.16 0)
+		(effects
+			(font
+				(size 1.27 1.27)
+			)
+			(justify left bottom)
+		)
+	)
+	(text "USB"
+		(exclude_from_sim no)
+		(at 40.005 187.325 0)
+		(effects
+			(font
+				(size 1.27 1.27)
+			)
+			(justify left bottom)
+		)
+	)
 	(junction
 		(at 107.95 62.23)
@@
 	)
 	(junction
-		(at 170.815 129.54)
-		(diameter 0)
-		(color 0 0 0 0)
-	)
-	(junction
 		(at 62.865 24.765)
 		(diameter 0)
@@
 	(wire
 		(pts
-			(xy 175.895 142.24) (xy 175.895 137.795)
-		)
-		(stroke
-			(width 0)
-			(type default)
-		)
-	)
-	(wire
-		(pts
 			(xy 247.65 33.02) (xy 238.76 33.02)
 		)
@@
 	(wire
 		(pts
-			(xy 175.895 129.54) (xy 175.895 130.175)
-		)
-		(stroke
-			(width 0)
-			(type default)
-		)
-	)
-	(wire
-		(pts
 			(xy 102.87 249.555) (xy 102.87 254)
 		)
@@
 	(wire
 		(pts
-			(xy 170.815 129.54) (xy 175.895 129.54)
-		)
-		(stroke
-			(width 0)
-			(type default)
-		)
-	)
-	(wire
-		(pts
 			(xy 160.02 258.445) (xy 169.545 258.445)
 		)
@@
 		)
 	)
-	(rectangle
-		(start 13.97 145.415)
-		(end 45.085 187.96)
-		(stroke
-			(width 0)
-			(type default)
-		)
-		(fill
-			(type none)
-		)
-	)
-	(rectangle
-		(start 13.97 13.97)
-		(end 194.31 187.96)
-		(stroke
-			(width 0.3)
-			(type default)
-		)
-		(fill
-			(type none)
-		)
-	)
-	(rectangle
-		(start 13.97 187.96)
-		(end 247.015 282.575)
-		(stroke
-			(width 0)
-			(type default)
-		)
-		(fill
-			(type none)
-		)
-	)
-	(rectangle
-		(start 13.97 122.555)
-		(end 45.085 145.415)
-		(stroke
-			(width 0)
-			(type default)
-		)
-		(fill
-			(type none)
-		)
-	)
-	(text "Flash\n"
-		(exclude_from_sim no)
-		(at 266.7 130.175 0)
-		(effects
-			(font
-				(size 1.27 1.27)
-			)
-			(justify left bottom)
-		)
-	)
-	(text "Meter0"
-		(exclude_from_sim no)
-		(at 257.175 65.405 0)
-		(effects
-			(font
-				(size 1.27 1.27)
-			)
-			(justify left bottom)
-		)
-	)
-	(text "Power "
-		(exclude_from_sim no)
-		(at 38.735 44.45 0)
-		(effects
-			(font
-				(size 1.27 1.27)
-			)
-			(justify left bottom)
-		)
-	)
-	(text "Crystal\n"
-		(exclude_from_sim no)
-		(at 36.83 144.78 0)
-		(effects
-			(font
-				(size 1.27 1.27)
-			)
-			(justify left bottom)
-		)
-	)
-	(text "IF Sonar: high means button got pressed\nELSE : low"
-		(exclude_from_sim no)
-		(at 115.57 198.12 0)
-		(effects
-			(font
-				(size 1.27 1.27)
-			)
-			(justify left bottom)
-		)
-	)
-	(text "Controller (RP2040 )\n"
-		(exclude_from_sim no)
-		(at 147.955 186.055 0)
-		(effects
-			(font
-				(face "KiCad Font")
-				(size 2.54 2.54)
-				(thickness 0.508)
-				(bold yes)
-			)
-			(justify left bottom)
-		)
-	)
-	(text "SCL1\n"
-		(exclude_from_sim no)
-		(at 151.13 139.7 0)
-		(effects
-			(font
-				(size 1.27 1.27)
-			)
-			(justify left bottom)
-		)
-	)
-	(text "SDA1"
-		(exclude_from_sim no)
-		(at 151.13 137.16 0)
-		(effects
-			(font
-				(size 1.27 1.27)
-			)
-			(justify left bottom)
-		)
-	)
-	(text "USB"
-		(exclude_from_sim no)
-		(at 40.005 187.325 0)
-		(effects
-			(font
-				(size 1.27 1.27)
-			)
-			(justify left bottom)
-		)
-	)
 	(label "MOTOR"
 		(at 175.26 104.14 180)
@@
 		)
 	)
-	(label "LED2"
-		(at 175.895 142.24 90)
-		(effects
-			(font
-				(size 1.27 1.27)
-			)
-			(justify left bottom)
-		)
-	)
 	(label "GTD-6"
 		(at 63.5 198.755 270)
@@
 	)
 	(symbol
-		(lib_id "Device:LED")
-		(at 175.895 133.985 90)
-		(unit 1)
-		(exclude_from_sim no)
-		(in_bom yes)
-		(on_board yes)
-		(dnp no)
-		(fields_autoplaced yes)
-		(property "Reference" "D6"
-			(at 179.07 134.9375 90)
-			(effects
-				(font
-					(size 1.27 1.27)
-				)
-				(justify right)
-			)
-		)
-		(property "Value" "LED"
-			(at 179.07 137.4775 90)
-			(effects
-				(font
-					(size 1.27 1.27)
-				)
-				(justify right)
-			)
-		)
-		(property "Footprint" "Diode_SMD:D_0603_1608Metric_Pad1.05x0.95mm_HandSolder"
-			(at 175.895 133.985 0)
-			(effects
-				(font
-					(size 1.27 1.27)
-				)
-				(hide yes)
-			)
-		)
-		(property "Datasheet" "~"
-			(at 175.895 133.985 0)
-			(effects
-				(font
-					(size 1.27 1.27)
-				)
-				(hide yes)
-			)
-		)
-		(property "Description" ""
-			(at 175.895 133.985 0)
-			(effects
-				(font
-					(size 1.27 1.27)
-				)
-				(hide yes)
-			)
-		)
-		(pin "1"
-		)
-		(pin "2"
-		)
-		(instances
-			(project "opsx_x"
-				(path "/b68e25c7-58ea-4fd3-9614-c4064fa4b280"
-					(reference "D6")
-					(unit 1)
-				)
-			)
-		)
-	)
-	(symbol
 		(lib_id "power:+3.3V")
 		(at 44.45 200.025 0)
@@
 		)
 	)
+	(embedded_fonts no)
 )
