File: Hardwares/MainController/rev2/opsx_x.kicad_sch (KiCad schematic)
At the start: 61 parts, among them J1 Conn_01x02, J3 Conn_01x02, Q1 Q_NMOS_GSD, Q2 Q_NMOS_GSD, Q3 Q_PMOS_GSD, Q4 MMBT3904, U1 RP2040, U2 TLV70433DBVR, U3 W25Q128JVS, U4 OPTICAL-TSL2561T(6P-3.8X2.6MM), Y1 Crystal_GND2

Commit message: 硬件更新：新增 Rev3_Normal 主板设计、FPC 柔性电路板、PowerBack 导光片壳体
- 新增 MainController Rev3_Normal (SX70z_Normal KiCad 工程 + Gerber + BOM)
- 新增 Fabrication BodyFPC 柔性电路板 Gerber
- 更新 MainController rev2 PCB
- 更新 PowerBack 外壳/快装板/导光片 (SLDPRT + STL + 3MF)

Co-Authored-By: Claude Opus 4.7 <noreply@anthropic.com>
Parts:
- added Q5: MMBT3904, Package_TO_SOT_SMD:SOT-23, symbol Transistor_BJT:MMBT3904
- added Q6: Q_PMOS_GSD, Package_TO_SOT_SMD:SOT-23, symbol Device:Q_PMOS_GSD
- added R26: 2.7k, Resistor_SMD:R_0402_1005Metric_Pad0.72x0.64mm_HandSolder, symbol Device:R
- added R7: 5.6k, Resistor_SMD:R_0402_1005Metric_Pad0.72x0.64mm_HandSolder, symbol Device:R
- added R8: 47k, Resistor_SMD:R_0402_1005Metric_Pad0.72x0.64mm_HandSolder, symbol Device:R
- added TP2: TestPoint, TestPoint:TestPoint_Pad_2.0x2.0mm, symbol Connector:TestPoint
- added Z4, Z5: ~, OPSX:Selector_default, symbol OPSX:selector_default
Connections:
- net +3.3V: now also Z5.3; no longer sx1.VO
- net GND: now also Q5.2 (E), R26.1, TP2.1
- net SCL1: now also Z4.3; no longer sx1.SCL
- net VCC: now also Q6.2 (S), R8.1, Z5.1
- net FF_Left_MCU: now reaches U1.18 (GPIO15)
- net FF_Left_MCU: now also R7.2
- new net: Q5.3 (C), Q6.1 (G), R8.2
- new net: Q5.1 (B), R7.1
- new net FF_Left: Q6.3 (D), R26.2, Z4.1
- new net FF_Left_Board: Z4.2, sx1.SCL
- new net VO_Left_Board: Z5.2, sx1.VO
- no-connect marks 16 -> 15
Other:
- note added: "SCL1(not sonnar)"
- note added: "SDA1(not sonnar)"
