File: Hardwares/PowerBack/sx70PowerPack/sx70battery.kicad_pcb (KiCad board)
At the start: 2 copper layers, 65 x 74 mm, 44 parts, among them J1 USB_C_Receptacle_PowerOnly_6P, U1 TP4057, U3 LN60A, U4 TPS61085DGK

Commit message: 外置电池设计完毕，生成光绘文件
Parts:
- C10: value 1uf -> 100nf
- C11: value 1uf -> 1nf
- R6: value 10k -> 8.2k
- R7: value 68k -> 69.8k
Routing:
- net GND: track 11.2 -> 11.6 mm, vias 75 -> 89
Other:
- board text added: "https://github.com/ZeshuLiu/SX-70-Mk2"

Commit message: 电池2.1版本（CC识别可以充电）
Parts:
- added R10: 5.1k, Resistor_SMD:R_0603_1608Metric_Pad0.98x0.95mm_HandSolder, F.Cu at (151.8, 115.6)
- added R11: 5.1k, Resistor_SMD:R_0603_1608Metric_Pad0.98x0.95mm_HandSolder, F.Cu at (148.1, 115.6)
Connections:
- J1 pad A5: unconnected-(J1-CC1-PadA5) -> Net-(J1-CC1)
- J1 pad B5: unconnected-(J1-CC2-PadB5) -> Net-(J1-CC2)
Routing:
- net Net-(J1-CC1): track 0.00 -> 3.10 mm
- net Net-(J1-CC2): track 0.00 -> 3.09 mm
- net GND: vias 89 -> 88

Commit message: 代码OK，电屁股正在做
Parts:
- removed C10: 100nf, Capacitor_SMD:C_0603_1608Metric_Pad1.08x0.95mm_HandSolder
- removed C11: 1nf, Capacitor_SMD:C_0603_1608Metric_Pad1.08x0.95mm_HandSolder
- removed C12, C8: 10uf, Capacitor_Tantalum_SMD:CP_EIA-3216-18_Kemet-A
- removed C13: 10uf, Capacitor_SMD:C_0805_2012Metric_Pad1.18x1.45mm_HandSolder
- removed C9: 1uf, Capacitor_SMD:C_0603_1608Metric_Pad1.08x0.95mm_HandSolder
- removed D6: B340A, Diode_SMD:D_SMA
- removed L2: 3.3uH, Inductor_SMD:L_Cenker_CKCS6020
- removed R6: 8.2k, Resistor_SMD:R_0603_1608Metric_Pad0.98x0.95mm_HandSolder
- removed R7: 69.8k, Resistor_SMD:R_0603_1608Metric_Pad0.98x0.95mm_HandSolder
- removed R8: 18k, Resistor_SMD:R_0603_1608Metric_Pad0.98x0.95mm_HandSolder
- removed U4: TPS61085DGK, Package_SO:VSSOP-8_3.0x3.0mm_P0.65mm
- added C3: 100nf, Capacitor_SMD:C_0603_1608Metric, F.Cu at (117.8, 86.0)
- added C4: 1uf, Capacitor_SMD:C_1206_3216Metric_Pad1.33x1.80mm_HandSolder, F.Cu at (120.2, 54.0)
- added C5: 10uf, Capacitor_SMD:C_1206_3216Metric_Pad1.33x1.80mm_HandSolder, F.Cu at (132.5, 55.2)
- added D1: SS34, Diode_SMD:D_SMA, F.Cu at (132.2, 58.2)
- added D7: 1N5819WS, Diode_SMD:D_SOD-323_HandSoldering, F.Cu at (132.5, 53.0)
- added L1: 4.7uH, Inductor_SMD:L_APV_APH0650, F.Cu at (123.8, 61.0)
- added R12: 100, Resistor_SMD:R_0603_1608Metric_Pad0.98x0.95mm_HandSolder, F.Cu at (114.0, 86.0)
- added R13: 1k, Resistor_SMD:R_0603_1608Metric_Pad0.98x0.95mm_HandSolder, F.Cu at (118.5, 83.2)
- added R15: 330k, Resistor_SMD:R_0603_1608Metric_Pad0.98x0.95mm_HandSolder, F.Cu at (127.7, 51.2)
- added R16: 51k, Resistor_SMD:R_0603_1608Metric_Pad0.98x0.95mm_HandSolder, F.Cu at (124.2, 51.2)
- added U2: DW01A, Package_TO_SOT_SMD:SOT-23-6, F.Cu at (115.8, 83.0)
- added U5: ~, Package_SO:TSSOP-8_4.4x3mm_P0.65mm, F.Cu at (115.8, 67.2)
- added U6: ~, Package_SO:TSSOP-8_4.4x3mm_P0.65mm, F.Cu at (115.8, 78.4)
- added U7: ~, Package_SO:TSSOP-8_4.4x3mm_P0.65mm, F.Cu at (115.8, 74.8)
- added U8: ~, Package_SO:TSSOP-8_4.4x3mm_P0.65mm, F.Cu at (115.8, 71.0)
- added U9: TLV61048DBVR, Package_TO_SOT_SMD:SOT-23-6, F.Cu at (125.5, 55.2)
- moved 6V+1 41.3 mm to (152.5, 55.2)
- moved GND2 41.3 mm to (156.2, 55.2)
- moved J1 24.4 mm to (130.5, 107.0)
- moved C7 11.7 mm to (117.6, 96.2)
- moved R2 11.7 mm to (120.6, 99.5)
- moved R3 11.7 mm to (125.3, 95.2)
- moved R4 11.7 mm to (125.3, 96.8)
- moved R5 11.7 mm to (125.3, 98.2)
- moved U3 11.7 mm to (121.1, 96.8)
- moved S1 11.5 mm to (110.2, 95.2)
- moved C1 11.2 mm to (112.5, 105.0)
- moved C2 11.2 mm to (115.2, 101.8)
- moved CHG1 11.2 mm to (109.5, 103.1)
- moved R1 11.2 mm to (119.2, 103.8)
- moved R9 11.2 mm to (116.5, 107.9)
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Connections:
- BAT-1 pad 1: GND -> /RealBat-
- U1 pad 2: GND -> /RealBat-
Routing:
- net /BAT+: track 100.5 -> 0.00 mm
- net +5V: track 43.9 -> 0.00 mm
- net Net-(D2-K): track 28.9 -> 0.00 mm
- net Net-(D5-K): track 28.3 -> 0.00 mm
- net +6V: track 59.1 -> 30.9 mm
- net Net-(D4-K): track 27.6 -> 0.00 mm
- net Net-(D3-K): track 27.6 -> 0.00 mm
- net Net-(CHG1-K): track 14.1 -> 0.00 mm
- net Net-(STB1-K): track 9.02 -> 0.00 mm
- net Net-(U4-SS): track 8.26 -> 0.00 mm, vias 2 -> 0
- net /RealBat+: track 7.52 -> 0.00 mm
- net GND: track 11.6 -> 17.6 mm, vias 88 -> 82
- net Net-(U4-FB): track 4.28 -> 0.00 mm
- net Net-(J1-CC1): track 3.10 -> 0.00 mm
- net Net-(J1-CC2): track 3.09 -> 0.00 mm
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- added copper zone on F.Cu, net /SW
- removed copper zone on F.Cu, net +5V
- removed copper zone on F.Cu, net +6V
- removed copper zone on F.Cu, net Net-(D6-A)
Other:
- board size 65 x 74 mm -> 72 x 79.5 mm

Commit message: 声纳工作正常
Parts:
- removed REF** (x2): OSHW-Logo_5.7x6mm_Copper, Symbol:OSHW-Logo_5.7x6mm_Copper
- added Bolt3: M3_BOLT, MountingHole:MountingHole_3.2mm_M3_Pad, F.Cu at (175.0, 110.5)
- added Bolt4: M3_BOLT, MountingHole:MountingHole_3.2mm_M3_Pad, F.Cu at (113.0, 110.5)
- added C10: 1uf, Capacitor_SMD:C_0603_1608Metric, F.Cu at (142.8, 60.0)
- added C11: 22nf, Capacitor_SMD:C_0603_1608Metric, F.Cu at (154.0, 52.5)
- added C12: 2nf, Capacitor_SMD:C_0603_1608Metric, F.Cu at (143.5, 50.0)
- added C13: 100nf, Capacitor_SMD:C_0603_1608Metric, F.Cu at (150.0, 50.0)
- added C6: 22uf, Capacitor_SMD:C_1206_3216Metric_Pad1.33x1.80mm_HandSolder, F.Cu at (157.5, 51.8)
- added C8: 100nf, Capacitor_SMD:C_0603_1608Metric, F.Cu at (155.5, 52.5)
- added C9: 47uf, Capacitor_SMD:C_1206_3216Metric_Pad1.33x1.80mm_HandSolder, F.Cu at (140.8, 59.0)
- added D6: SS34, Diode_SMD:D_SMA, F.Cu at (148.5, 60.8)
- added L2: 3.3uH, Inductor_SMD:L_APV_APH0650, F.Cu at (157.5, 59.0)
- added R14: 866, Resistor_SMD:R_0603_1608Metric_Pad0.98x0.95mm_HandSolder, F.Cu at (146.8, 50.0)
- added R6: 39k, Resistor_SMD:R_0603_1608Metric_Pad0.98x0.95mm_HandSolder, F.Cu at (141.2, 53.0)
- added R7: 10k, Resistor_SMD:R_0603_1608Metric_Pad0.98x0.95mm_HandSolder, F.Cu at (141.2, 51.5)
- added R8: 60.4k, Resistor_SMD:R_0603_1608Metric_Pad0.98x0.95mm_HandSolder, F.Cu at (141.3, 54.5)
- added U4: ~, Package_SO:HTSSOP-14-1EP_4.4x5mm_P0.65mm_EP3.4x5mm_Mask3x3.1mm, F.Cu at (148.2, 54.8)
- Sx70_Pogopin1: footprint Jimmy_Library:sx_70_pogopin -> KiCadLib:sx_70_pogopin_phi2mm
- moved STB1 19.8 mm to (129.2, 106.5), turned to -90 degrees
- moved C3 19.5 mm to (113.7, 66.9), turned to 180 degrees
- moved R12 19.3 mm to (117.0, 66.9), turned to 180 degrees
- moved R9 18.8 mm to (131.5, 96.5), turned to 0 degrees
- moved R10 18.5 mm to (138.0, 103.2), turned to -90 degrees
- moved U5 18.4 mm to (115.7, 85.7), turned to 0 degrees
- moved CHG1 17.3 mm to (126.5, 106.5)
- moved R11 17.1 mm to (136.2, 103.2), turned to -90 degrees
- moved C1 16.8 mm to (128.0, 98.5), turned to 180 degrees
- moved R1 16.0 mm to (131.5, 93.5)
- moved R_PRG1 16.0 mm to (131.5, 95.0)
- moved U1 16.0 mm to (128.0, 94.8)
- moved C2 15.8 mm to (127.2, 91.5)
- moved 6V+1 15.2 mm to (137.5, 53.0), turned to 0 degrees
- moved U2 13.1 mm to (115.7, 69.9), turned to 90 degrees
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Connections:
- C2 pad 1: /BAT+ -> /RealBat+
- U1 pad 2: /RealBat- -> GND
- U1 pad 3: /BAT+ -> /RealBat+
- U5 pad 1: Net-(U5-S2) -> unconnected-(U5-D1-Pad1)
- U5 pad 8: Net-(U5-S2) -> unconnected-(U5-D2-Pad8)
- U6 pad 1: Net-(U6-D1) -> unconnected-(U6-D1-Pad1)
- U6 pad 8: Net-(U6-D1) -> unconnected-(U6-D2-Pad8)
- U7 pad 1: Net-(U7-D1) -> unconnected-(U7-D1-Pad1)
- U7 pad 8: Net-(U7-D1) -> unconnected-(U7-D2-Pad8)
- U8 pad 1: Net-(U8-D1) -> unconnected-(U8-D1-Pad1)
- U8 pad 8: Net-(U8-D1) -> unconnected-(U8-D2-Pad8)
Routing:
- net /BAT+: track 0.00 -> 78.7 mm, vias 4 -> 14
- net /RealBat+: track 0.00 -> 46.7 mm, vias 0 -> 2
- net +5V: track 0.00 -> 39.0 mm
- net Net-(U2-OD): track 0.00 -> 27.1 mm
- net Net-(U2-OC): track 0.00 -> 24.0 mm
- net GND: track 17.6 -> 37.1 mm, vias 82 -> 175
- net Net-(D5-K): track 0.00 -> 18.3 mm, vias 2 -> 0
- net Net-(CHG1-K): track 0.00 -> 14.4 mm, vias 2 -> 0
- net Net-(D4-K): track 0.00 -> 13.6 mm, vias 2 -> 0
- net Net-(D2-K): track 0.00 -> 11.0 mm, vias 2 -> 0
- net Net-(D3-K): track 0.00 -> 10.7 mm, vias 2 -> 0
- net Net-(STB1-K): track 0.00 -> 10.3 mm, vias 2 -> 0
- net +6V: track 30.9 -> 20.9 mm, vias 2 -> 0
- net Net-(U4-FB): track 0.00 -> 5.52 mm
- net Net-(U4-COMP): track 0.00 -> 5.35 mm
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- added copper zone on F.Cu, net +6V
- added copper zone on B.Cu, net /BAT+
- added copper zone on F.Cu, net /RealBat-
- added copper zone on F.Cu, net Net-(D6-A)
Other:
- board size 72 x 79.5 mm -> 72 x 68.5 mm
