File: Hardwares/MainController/Rev3_Normal/SX70z_Normal/SX70z_Normal.kicad_sch (KiCad schematic)
At the start: 50 parts, among them J1 Conn_01x02, J2 Conn_01x03_Socket, J3 Conn_01x02, Q1 Q_NMOS_GSD, Q2 Q_NMOS_GSD, Q5 MMBT3904, Q6 Q_PMOS_GSD, U3 SPX3819M5-L-3-3, U4 ESP32-PICO-D4, U5 OPT4001DTSR

Commit message: 修改SX70zPCB的小问题，投产机身控制器
Parts:
- added C8: 10uf, Capacitor_SMD:C_0402_1005Metric, symbol Device:C
- added R15: 10k, Resistor_SMD:R_0402_1005Metric_Pad0.72x0.64mm_HandSolder, symbol Device:R
Connections:
- net +3.3V: now also R15.2
- net BOOT: now also R15.1
- net EN: now also C8.2
- net GND: now also C8.1
Other:
- moved on the sheet: R4
